File: PCB/board.brd (EAGLE design)
At the start: 49.5 x 100 mm, 64 parts, among them IC1 LM2596S, J1 MICRO-SD_CARD_SOCKETTINY, J12 AVR_SPI_PROG_3X2NS, Q1 220mA/50V/3.5Ω, Q2 220mA/50V/3.5Ω, U2 ESP-WROOM-02, U3 ATMEGA328P_TQFP, U4 PC817X2NIP0F, U5 INFINEON_BTS7960BINFINEON_BTS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, U6 INFINEON_BTS7960BINFINEON_BTS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

Commit message: update
Parts:
- R1, R2, R3, R4: value (none) -> 1k
- R5: value (none) -> 1M
- moved R4 18.9 mm to (12.8, 10.0), turned to 0 degrees
Connections:
- removed net N$6: R4.2, S3.3, S3.4
- net 5V: no longer R2.1, R3.1, R4.1
- net GND: now also R4.2, S3.3, S3.4
- net N$3: now also R2.2, R3.1, S2.3, S2.4; no longer R1.2, S4.3, S4.4
- net N$4: now also R3.2, R4.1, S1.3, S1.4; no longer R2.2, S2.3, S2.4
- net N$5: now also R1.2, R2.1, S4.3, S4.4; no longer R3.2, S1.3, S1.4
Routing:
- net N$6: track 13.9 -> 0.00 mm
- net N$5: track 9.35 -> 23.0 mm
- net N$4: track 9.54 -> 23.1 mm, vias 0 -> 2
- net 5V: track 159.6 -> 151.0 mm, vias 6 -> 7
- net N$3: track 9.10 -> 15.0 mm
- net GND: track 0.00 -> 5.59 mm
