File: PCB/board.sch (EAGLE design)
At the start: 64 parts, among them IC1 LM2596S, J1 MICRO-SD_CARD_SOCKETTINY, J12 AVR_SPI_PROG_3X2NS, Q1 220mA/50V/3.5Ω, Q2 220mA/50V/3.5Ω, U2 ESP-WROOM-02, U3 ATMEGA328P_TQFP, U4 PC817X2NIP0F, U5 INFINEON_BTS7960BINFINEON_BTS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, U6 INFINEON_BTS7960BINFINEON_BTS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

Commit message: update
Parts:
- R1, R2, R3, R4: value (none) -> 1k
- R5: value (none) -> 1M
Connections:
- removed net N$6: R4.2, S3.2
- net 5V: no longer R2.1, R3.1, R4.1
- net GND: now also R4.2, S3.2
- net N$3: now also R2.2, R3.1, S2.2; no longer R1.2, S4.2
- net N$4: now also R3.2, R4.1, S1.2; no longer R2.2, S2.2
- net N$5: now also R1.2, R2.1, S4.2; no longer R3.2, S1.2
Other:
- moved on the sheet: R1, R2, R3, R4
